Commit message: cameras fixed in position and orientation

File: box_urdf/urdf/camera_box_RGB.urdf (robot description, URDF)
Before this commit: robot test_model, 2 links, 1 joints
Joints:
- joint object_base_joint: origin xyz=0 0 0 rpy=0 -1.51 0 -> xyz=0 0 0 rpy=0 1.05 0

Commit message: Panels detection fixed

File: box_urdf/urdf/camera_box_RGB.urdf (robot description, URDF)
Before this commit: robot test_model, 2 links, 1 joints
Joints:
- joint object_base_joint: origin xyz=0 0 0 rpy=0 1.05 0 -> xyz=0 0 0 rpy=0 1.57 0
